Commit message: improved pick place

File: my_robot/my_robot_description/urdf/my_robot.urdf.xacro (robot description, xacro)
@@ -22,3 +22,10 @@
     <origin xyz="0 0 0.05" rpy="0 0 0" />
   </xacro:rail>
+  <!--Floor-->
+  <xacro:include filename="$(find my_robot_description)/urdf/floor.xacro" />
+  <xacro:floor prefix="" parent="world" >
+    <origin xyz="0 -0.85 0" rpy="0 0 0" />
+  </xacro:floor>
+  <!--Materials-->
+  <xacro:include filename="$(find my_robot_description)/urdf/materials.xacro" />
 </robot>

File: my_robot/my_robot_description/urdf/rail.xacro (robot description, xacro)
@@ -17,4 +17,5 @@
                 <box size="${rail_size_x} ${rail_size_y} ${rail_size_z}" />
             </geometry>
+            <material name="grey"/>
         </visual>
         <collision>
@@ -43,4 +44,5 @@
                 <box size="${platform_size_x} ${platform_size_y} ${platform_size_z}" />
             </geometry>
+            <material name="dark_grey"/>
         </visual>
         <collision>
@@ -68,5 +70,5 @@
         <child link="${prefix}base_platform_link"/>
         <axis xyz="1 0 0 "/>
-        <limit lower="${-1*rail_size_x/2}" upper="${rail_size_x/2}" effort="100" velocity="1.0"/>
+        <limit lower="${-1*rail_size_x/2}" upper="${rail_size_x/2}" effort="1000" velocity="2.0"/>
     </joint>
     <joint name="${prefix}platform_joint" type="fixed">

Commit message: [CleanUp] Refactor and clean up robot model and moveit files

File: my_robot/my_robot_description/urdf/my_robot.urdf.xacro (robot description, xacro)
@@ -3,18 +3,8 @@
        name="ur10" >
   <xacro:arg name="transmission_hw_interface" default="hardware_interface/PositionJointInterface"/>
-  <!-- common stuff -->
-  <xacro:include filename="$(find ur_description)/urdf/common.gazebo.xacro" />
   <!-- ur10 -->
-  <xacro:include filename="$(find ur_description)/urdf/ur10.urdf.xacro" />
-  <!-- arm -->
-  <xacro:ur10_robot prefix="" joint_limited="false"
-    transmission_hw_interface="$(arg transmission_hw_interface)"
-  />
+  <xacro:include filename="$(find ur_description)/urdf/ur10.xacro" />
+  <!-- world -->
   <link name="world" />
-  <!-- <joint name="world_joint" type="fixed">
-    <parent link="world" />
-    <child link = "base_link" />
-    <origin xyz="0.0 0.0 0.0" rpy="0.0 0.0 0.0" />
-  </joint> -->
   <!-- rail -->
   <xacro:include filename="$(find my_robot_description)/urdf/rail.xacro" />
